File: kicad/cool936.sch (KiCad schematic (older format))
At the start: 84 parts, among them J12 MJ-4PP-9, J13 MJ-4PP-9, SW1 Switch_SW_Push, SW10 Switch_SW_Push, SW101 Switch_SW_Push, SW102 Switch_SW_Push, SW103 Switch_SW_Push, SW11 Switch_SW_Push, SW12 Switch_SW_Push, SW13 Switch_SW_Push, SW14 Switch_SW_Push, SW15 Switch_SW_Push, SW16 Switch_SW_Push, SW17 Switch_SW_Push, SW18 Switch_SW_Push, SW19 Switch_SW_Push, SW2 Switch_SW_Push, SW20 Switch_SW_Push, SW201 Switch_SW_Push, SW21 Switch_SW_Push, SW22 Switch_SW_Push, SW23 Switch_SW_Push, SW24 Switch_SW_Push, SW25 Switch_SW_Push, SW26 Switch_SW_Push, SW27 Switch_SW_Push, SW28 Switch_SW_Push, SW29 Switch_SW_Push, SW3 Switch_SW_Push, SW30 Switch_SW_Push, SW301 Switch_SW_Push, SW302 Switch_SW_Push, SW303 Switch_SW_Push, SW4 Switch_SW_Push, SW5 Switch_SW_Push, SW6 Switch_SW_Push, SW7 Switch_SW_Push, SW8 Switch_SW_Push, SW900 SW_PUSH, SW901 SW_PUSH, U1 ProMicro, U2 ProMicro

Commit message: 修正
Parts:
- U1, U2: footprint logo:ProMicro_v3_kimura -> logo:ProMicro_v3_kimura_for_cool936; symbol kbd:ProMicro -> cool936-rescue:ProMicro-kbd
Changed lines of the file:
@@
 	3075 5225 3675 5225
 $Comp
-L kbd:ProMicro U1
+L cool936-rescue:ProMicro-kbd U1
 U 1 1 62079521
 P 3025 1600
 F 0 "U1" H 3025 2637 60  0000 C CNN
 F 1 "ProMicro" H 3025 2531 60  0000 C CNN
-F 2 "logo:ProMicro_v3_kimura" H 3125 550 60  0001 C CNN
+F 2 "logo:ProMicro_v3_kimura_for_cool936" H 3125 550 60  0001 C CNN
 F 3 "" H 3125 550 60  0000 C CNN
 	1    3025 1600
@@
 Text GLabel 2325 1750 0    50   Input ~ 0
 col3L
-Text GLabel 2325 1850 0    50   Input ~ 0
+Text GLabel 2325 1950 0    50   Input ~ 0
 col4L
 Text GLabel 3725 1450 2    50   Input ~ 0
@@
 Text GLabel 3725 1650 2    50   Input ~ 0
 row2L
-Text GLabel 3725 1750 2    50   Input ~ 0
+Text GLabel 3725 1850 2    50   Input ~ 0
 row3L
 Text GLabel 2325 850  0    50   Input ~ 0
@@
 NoConn ~ 3725 1250
 NoConn ~ 3725 1350
-NoConn ~ 3725 1850
+NoConn ~ 3725 1750
 NoConn ~ 3725 1950
-NoConn ~ 2325 1950
+NoConn ~ 2325 1850
 NoConn ~ 2325 1350
 NoConn ~ 2325 1250
@@
 	1675 1725 1525 1725
 $Comp
-L kbd:ProMicro U2
+L cool936-rescue:ProMicro-kbd U2
 U 1 1 621A5C74
 P 7025 1600
 F 0 "U2" H 7025 2637 60  0000 C CNN
 F 1 "ProMicro" H 7025 2531 60  0000 C CNN
-F 2 "logo:ProMicro_v3_kimura" H 7125 550 60  0001 C CNN
+F 2 "logo:ProMicro_v3_kimura_for_cool936" H 7125 550 60  0001 C CNN
 F 3 "" H 7125 550 60  0000 C CNN
 	1    7025 1600
@@
 Text GLabel 6325 1750 0    50   Input ~ 0
 col3R
-Text GLabel 6325 1850 0    50   Input ~ 0
+Text GLabel 6325 1950 0    50   Input ~ 0
 col4R
 Text GLabel 7725 1450 2    50   Input ~ 0
@@
 Text GLabel 7725 1650 2    50   Input ~ 0
 row2R
-Text GLabel 7725 1750 2    50   Input ~ 0
+Text GLabel 7725 1850 2    50   Input ~ 0
 row3R
 Text GLabel 6325 850  0    50   Input ~ 0
@@
 NoConn ~ 7725 1250
 NoConn ~ 7725 1350
-NoConn ~ 7725 1850
+NoConn ~ 7725 1750
 NoConn ~ 7725 1950
-NoConn ~ 6325 1950
+NoConn ~ 6325 1850
 NoConn ~ 6325 1350
 NoConn ~ 6325 1250

Commit message: fix
Parts:
- added J1, J2: Conn_01x03, kbd:StripLED_1side, symbol Connector_Generic:Conn_01x03
- L1, L2, L3, L4, L5, L6: footprint KiCAD_FootPrint-master:YS-SK6812MINI-E_UG -> kbd:LED_WS2812B-PLCC4
- SW1, SW10, SW101, SW102, SW103, SW11, SW12, SW13, SW14, SW15, SW16, SW17, SW18, SW19, SW2, SW20, SW201, SW21, SW22, SW23, SW24, SW25, SW26, SW27, SW28, SW29, SW3, SW30, SW301, SW302, SW303, SW4, SW5, SW6, SW7, SW8: footprint kbd:CherryMX-Hotswap-v2 -> logo:CherryMX_Hotswap_kimura
Connections:
- net GND: now also J1.1 (Pin_1), J2.1 (Pin_1)
- net LEDL: now also J1.2 (Pin_2)
- net LEDR: now also J2.2 (Pin_2)
- net VCC: now also J1.3 (Pin_3), J2.3 (Pin_3)

Commit message: fix
Parts:
- removed L1, L2, L3, L4, L5, L6: SK6812MINI, kbd:LED_WS2812B-PLCC4, symbol kbd:SK6812MINI
Connections:
- no-connect marks 20 -> 18
Other:
- moved on the sheet: J2
Changed lines of the file:
@@
-	1    0    0    -1
-$EndComp
-$Comp
-L kbd:SK6812MINI L3
-U 1 1 620F8884
-P 2200 5925
-F 0 "L3" H 2200 6187 51  0000 C CNN
-F 1 "SK6812MINI" H 2200 6122 16  0000 C CNN
-F 2 "kbd:LED_WS2812B-PLCC4" H 2200 5925 60  0001 C CNN
-F 3 "" H 2200 5925 60  0001 C CNN
-	1    2200 5925
-	1    0    0    -1
-$EndComp
-$Comp
-L kbd:SK6812MINI L2
-U 1 1 620F8C84
-P 2750 5925
-F 0 "L2" H 2750 6187 51  0000 C CNN
-F 1 "SK6812MINI" H 2750 6122 16  0000 C CNN
-F 2 "kbd:LED_WS2812B-PLCC4" H 2750 5925 60  0001 C CNN
-F 3 "" H 2750 5925 60  0001 C CNN
-	1    2750 5925
-	1    0    0    -1
-$EndComp
-$Comp
-L kbd:SK6812MINI L1
-U 1 1 620F9E3C
-P 3300 5925
-F 0 "L1" H 3300 6187 51  0000 C CNN
-F 1 "SK6812MINI" H 3300 6122 16  0000 C CNN
-F 2 "kbd:LED_WS2812B-PLCC4" H 3300 5925 60  0001 C CNN
-F 3 "" H 3300 5925 60  0001 C CNN
-	1    3300 5925
 	1    0    0    -1
 $EndComp
@@
 	2325 1150 1850 1150
 Connection ~ 1850 1150
-Wire Wire Line
-	3100 5825 3025 5825
-Wire Wire Line
-	3025 5825 3025 6025
-Wire Wire Line
-	3025 6025 2950 6025
-Wire Wire Line
-	2550 5825 2475 5825
-Wire Wire Line
-	2475 5825 2475 6025
-Wire Wire Line
-	2475 6025 2400 6025
-Wire Wire Line
-	3100 6025 3100 6125
-Wire Wire Line
-	3100 6125 2550 6125
-Wire Wire Line
-	2550 6125 2550 6025
-Wire Wire Line
-	2550 6125 2000 6125
-Wire Wire Line
-	2000 6125 2000 6025
-Connection ~ 2550 6125
-$Comp
-L power:VCC #PWR0107
-U 1 1 621604DA
-P 1925 5575
-F 0 "#PWR0107" H 1925 5425 50  0001 C CNN
-F 1 "VCC" H 1940 5748 50  0000 C CNN
-F 2 "" H 1925 5575 50  0001 C CNN
-F 3 "" H 1925 5575 50  0001 C CNN
-	1    1925 5575
-	1    0    0    -1
-$EndComp
-Wire Wire Line
-	1925 6125 2000 6125
-Connection ~ 2000 6125
-Wire Wire Line
-	2400 5825 2400 5575
-Wire Wire Line
-	2400 5575 1925 5575
-Wire Wire Line
-	2400 5575 2950 5575
-Wire Wire Line
-	2950 5575 2950 5825
-Connection ~ 2400 5575
-Wire Wire Line
-	2950 5575 3500 5575
-Wire Wire Line
-	3500 5575 3500 5825
-Connection ~ 2950 5575
-$Comp
-L power:GND #PWR0108
-U 1 1 6216C4D9
-P 1925 6125
-F 0 "#PWR0108" H 1925 5875 50  0001 C CNN
-F 1 "GND" H 1930 5952 50  0000 C CNN
-F 2 "" H 1925 6125 50  0001 C CNN
-F 3 "" H 1925 6125 50  0001 C CNN
-	1    1925 6125
-	1    0    0    -1
-$EndComp
-NoConn ~ 2000 5825
-Text GLabel 3500 6025 2    50   Input ~ 0
-LEDL
 Text GLabel 2325 950  0    50   Input ~ 0
 DataL
@@
 	5675 1725 5525 1725
 $Comp
-L kbd:SK6812MINI L6
-U 1 1 621B08CC
-P 6150 5925
-F 0 "L6" H 6150 6187 51  0000 C CNN
-F 1 "SK6812MINI" H 6150 6122 16  0000 C CNN
-F 2 "kbd:LED_WS2812B-PLCC4" H 6150 5925 60  0001 C CNN
-F 3 "" H 6150 5925 60  0001 C CNN
-	1    6150 5925
-	1    0    0    -1
-$EndComp
-$Comp
-L kbd:SK6812MINI L5
-U 1 1 621B08D6
-P 6700 5925
-F 0 "L5" H 6700 6187 51  0000 C CNN
-F 1 "SK6812MINI" H 6700 6122 16  0000 C CNN
-F 2 "kbd:LED_WS2812B-PLCC4" H 6700 5925 60  0001 C CNN
-F 3 "" H 6700 5925 60  0001 C CNN
-	1    6700 5925
-	1    0    0    -1
-$EndComp
-$Comp
-L kbd:SK6812MINI L4
-U 1 1 621B08E0
-P 7250 5925
-F 0 "L4" H 7250 6187 51  0000 C CNN
-F 1 "SK6812MINI" H 7250 6122 16  0000 C CNN
-F 2 "kbd:LED_WS2812B-PLCC4" H 7250 5925 60  0001 C CNN
-F 3 "" H 7250 5925 60  0001 C CNN
-	1    7250 5925
-	1    0    0    -1
-$EndComp
-Wire Wire Line
-	7050 5825 6975 5825
-Wire Wire Line
-	6975 5825 6975 6025
-Wire Wire Line
-	6975 6025 6900 6025
-Wire Wire Line
-	6500 5825 6425 5825
-Wire Wire Line
-	6425 5825 6425 6025
-Wire Wire Line
-	6425 6025 6350 6025
-Wire Wire Line
-	7050 6025 7050 6125
-Wire Wire Line
-	7050 6125 6500 6125
-Wire Wire Line
-	6500 6125 6500 6025
-Wire Wire Line
-	6500 6125 5950 6125
-Wire Wire Line
-	5950 6125 5950 6025
-Connection ~ 6500 6125
-$Comp
-L power:VCC #PWR0121
-U 1 1 621B08F6
-P 5875 5575
-F 0 "#PWR0121" H 5875 5425 50  0001 C CNN
-F 1 "VCC" H 5890 5748 50  0000 C CNN
-F 2 "" H 5875 5575 50  0001 C CNN
-F 3 "" H 5875 5575 50  0001 C CNN
-	1    5875 5575
-	1    0    0    -1
-$EndComp
-Wire Wire Line
-	5875 6125 5950 6125
-Connection ~ 5950 6125
-Wire Wire Line
-	6350 5825 6350 5575
-Wire Wire Line
-	6350 5575 5875 5575
-Wire Wire Line
-	6350 5575 6900 5575
-Wire Wire Line
-	6900 5575 6900 5825
-Connection ~ 6350 5575
-Wire Wire Line
-	6900 5575 7450 5575
-Wire Wire Line
-	7450 5575 7450 5825
-Connection ~ 6900 5575
-$Comp
-L power:GND #PWR0122
-U 1 1 621B090A
-P 5875 6125
-F 0 "#PWR0122" H 5875 5875 50  0001 C CNN
-F 1 "GND" H 5880 5952 50  0000 C CNN
-F 2 "" H 5875 6125 50  0001 C CNN
-F 3 "" H 5875 6125 50  0001 C CNN
-	1    5875 6125
-	1    0    0    -1
-$EndComp
-NoConn ~ 5950 5825
-$Comp
 L kbd:SW_PUSH SW900
 U 1 1 621B99DB
@@
 Text GLabel 7950 2100 0    50   Input ~ 0
 resetR
-Text GLabel 7450 6025 2    50   Input ~ 0
-LEDR
 $Comp
 L Connector_Generic:Conn_01x03 J2
 U 1 1 62754230
-P 7275 6375
-F 0 "J2" H 7193 6050 50  0000 C CNN
-F 1 "Conn_01x03" H 7193 6141 50  0000 C CNN
-F 2 "kbd:StripLED_1side" H 7275 6375 50  0001 C CNN
-F 3 "~" H 7275 6375 50  0001 C CNN
-	1    7275 6375
+P 8400 1550
+F 0 "J2" H 8318 1225 50  0000 C CNN
+F 1 "Conn_01x03" H 8318 1316 50  0000 C CNN
+F 2 "kbd:StripLED_1side" H 8400 1550 50  0001 C CNN
+F 3 "~" H 8400 1550 50  0001 C CNN
+	1    8400 1550
 	-1   0    0    1
 $EndComp
-Text GLabel 7475 6375 2    50   Input ~ 0
+Text GLabel 8600 1550 2    50   Input ~ 0
 LEDR
 $Comp
 L power:VCC #PWR0101
 U 1 1 62756F03
-P 7725 6275
-F 0 "#PWR0101" H 7725 6125 50  0001 C CNN
-F 1 "VCC" H 7740 6448 50  0000 C CNN
-F 2 "" H 7725 6275 50  0001 C CNN
-F 3 "" H 7725 6275 50  0001 C CNN
-	1    7725 6275
+P 8850 1450
+F 0 "#PWR0101" H 8850 1300 50  0001 C CNN
+F 1 "VCC" H 8865 1623 50  0000 C CNN
+F 2 "" H 8850 1450 50  0001 C CNN
+F 3 "" H 8850 1450 50  0001 C CNN
+	1    8850 1450
 	1    0    0    -1
 $EndComp
@@
 L power:GND #PWR0102
 U 1 1 627578A9
-P 7725 6475
-F 0 "#PWR0102" H 7725 6225 50  0001 C CNN
-F 1 "GND" H 7730 6302 50  0000 C CNN
-F 2 "" H 7725 6475 50  0001 C CNN
-F 3 "" H 7725 6475 50  0001 C CNN
-	1    7725 6475
-	1    0    0    -1
-$EndComp
-Wire Wire Line
-	7725 6275 7475 6275
-Wire Wire Line
-	7475 6475 7725 6475
+P 8850 1650
+F 0 "#PWR0102" H 8850 1400 50  0001 C CNN
+F 1 "GND" H 8855 1477 50  0000 C CNN
+F 2 "" H 8850 1650 50  0001 C CNN
+F 3 "" H 8850 1650 50  0001 C CNN
+	1    8850 1650
+	1    0    0    -1
+$EndComp
+Wire Wire Line
+	8850 1450 8600 1450
+Wire Wire Line
+	8600 1650 8850 1650
 $Comp
 L Connector_Generic:Conn_01x03 J1
