File: kicad/cool936.kicad_pcb (KiCad board)
At the start: 2 copper layers, 260.6 x 193.1 mm, 88 parts, among them J12 MJ-4PP-9, J13 MJ-4PP-9, SW1 Switch_SW_Push, SW10 Switch_SW_Push, SW101 Switch_SW_Push, SW102 Switch_SW_Push, SW103 Switch_SW_Push, SW11 Switch_SW_Push, SW12 Switch_SW_Push, SW13 Switch_SW_Push, SW14 Switch_SW_Push, SW15 Switch_SW_Push, SW16 Switch_SW_Push, SW17 Switch_SW_Push, SW18 Switch_SW_Push, SW19 Switch_SW_Push, SW2 Switch_SW_Push, SW20 Switch_SW_Push, SW201 Switch_SW_Push, SW21 Switch_SW_Push, SW22 Switch_SW_Push, SW23 Switch_SW_Push, SW24 Switch_SW_Push, SW25 Switch_SW_Push, SW26 Switch_SW_Push, SW27 Switch_SW_Push, SW28 Switch_SW_Push, SW29 Switch_SW_Push, SW3 Switch_SW_Push, SW30 Switch_SW_Push, SW301 Switch_SW_Push, SW302 Switch_SW_Push, SW303 Switch_SW_Push, SW4 Switch_SW_Push, SW5 Switch_SW_Push, SW6 Switch_SW_Push, SW7 Switch_SW_Push, SW8 Switch_SW_Push, SW900 SW_PUSH, SW901 SW_PUSH, U1 ProMicro, U2 ProMicro

Commit message: 修正
Parts:
- U1, U2: footprint logo:ProMicro_v3_kimura -> logo:ProMicro_v3_kimura_for_cool936
- moved U1 2.67 mm to (37.7, -0.38)
- moved U2 2.52 mm to (251.5, -0.41)
- moved D1 0.24 mm to (36.9, 1.34)
Connections:
- U1 pad 11: col4L -> Net-(U1-Pad11)
- U1 pad 12: Net-(U1-Pad12) -> col4L
- U1 pad 14: Net-(U1-Pad14) -> row3L
- U1 pad 15: row3L -> Net-(U1-Pad15)
- U2 pad 11: col4R -> Net-(U2-Pad11)
- U2 pad 12: Net-(U2-Pad12) -> col4R
- U2 pad 14: Net-(U2-Pad14) -> row3R
- U2 pad 15: row3R -> Net-(U2-Pad15)
Routing:
- net row3R: track 180.7 -> 238.8 mm, vias 0 -> 5
- net row2R: track 167.5 -> 147.3 mm, vias 1 -> 4
- net DataL: track 46.2 -> 60.2 mm
- net col0L: track 101.1 -> 109.6 mm, vias 0 -> 2
- net Net-(D1-Pad2): track 11.2 -> 16.1 mm
- net row0L: track 83.3 -> 86.7 mm
- net col4L: track 112.2 -> 109.1 mm
- net GND: track 333.3 -> 336.4 mm
- net row3L: track 125.7 -> 128.7 mm
- net col4R: track 65.8 -> 68.3 mm, vias 3 -> 4
- net VCC: track 289.1 -> 291.0 mm
- net resetL: track 71.7 -> 72.8 mm
- net row2L: track 131.2 -> 132.3 mm
- net LEDL: track 110.7 -> 111.6 mm
- net resetR: track 62.0 -> 61.0 mm, vias 2 -> 0
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Other:
- board text added: "cool936 designed by m.ki date 20220306 ver.1.1"
- board text removed: "cool936 designed by m.ki date 20220220 ver.1.0"

Commit message: fix
Routing:
- net LEDR: track 86.8 -> 86.3 mm

Commit message: fix
Parts:
- added J1: Conn_01x03, kbd:StripLED_1side, B.Cu at (113.6, 29.0)
- added J2: Conn_01x03, kbd:StripLED_1side, B.Cu at (190.2, 23.4)
- L1, L2, L3, L4, L5, L6: footprint KiCAD_FootPrint-master:YS-SK6812MINI-E_UG -> kbd:LED_WS2812B-PLCC4
- SW1, SW10, SW101, SW102, SW103, SW11, SW12, SW13, SW14, SW15, SW16, SW17, SW18, SW19, SW2, SW20, SW201, SW21, SW22, SW23, SW24, SW25, SW26, SW27, SW28, SW29, SW3, SW30, SW301, SW302, SW303, SW4, SW5, SW6, SW7, SW8: footprint kbd:CherryMX-Hotswap-v2 -> logo:CherryMX_Hotswap_kimura
- moved D18 18.4 mm to (251.4, 15.5)
- moved G*** 14.9 mm to (71.1, 28.9)
- moved D19 10.0 mm to (267.8, 35.8), turned to 90 degrees
- moved G*** 9.98 mm to (222.4, 30.0)
- moved D11 6.89 mm to (60.8, 14.6)
- moved D102 6.87 mm to (39.4, 14.5)
- moved D12 6.69 mm to (79.7, 14.7)
- moved D17 6.35 mm to (232.6, 16.6)
- moved D16 4.97 mm to (213.5, 16.5)
- moved D15 4.52 mm to (194.3, 16.7)
- moved L4 4.09 mm to (198.4, 25.9)
- moved L2 2.86 mm to (71.5, 25.7)
- moved L3 2.85 mm to (45.1, 25.7)
- moved L1 2.80 mm to (100.0, 25.8)
- moved L6 2.76 mm to (249.7, 25.7)
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Routing:
- net row3R: track 238.8 -> 183.1 mm
- net GND: track 336.4 -> 382.1 mm
- net col3R: track 82.7 -> 108.2 mm
- net VCC: track 291.0 -> 313.9 mm, vias 8 -> 7
- net row1R: track 130.3 -> 147.4 mm
- net Net-(L4-Pad1): track 48.3 -> 32.2 mm, vias 2 -> 0
- net LEDR: track 86.3 -> 102.2 mm, vias 2 -> 1
- net col0R: track 157.0 -> 142.8 mm
- net col2R: track 122.9 -> 113.1 mm
- net row2R: track 147.3 -> 156.7 mm
- net LEDL: track 111.6 -> 120.0 mm, vias 0 -> 2
- net Net-(L5-Pad1): track 40.8 -> 32.6 mm
- net Net-(D18-Pad2): track 30.4 -> 22.4 mm
- net Net-(D26-Pad2): track 17.2 -> 9.75 mm
- net col1R: track 134.9 -> 128.3 mm
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Other:
- board text added: "cool936 designed by m.ki date 20220503 ver.1.3"
- board text removed: "cool936 designed by m.ki date 20220306 ver.1.1"

Commit message: fix
Parts:
- removed G***: LOGO, logo:dragonbreath_left
- removed G***: LOGO, logo:dragonbreath
- removed L1, L2, L3, L4, L5, L6: SK6812MINI, kbd:LED_WS2812B-PLCC4
- removed kiritori (x2): kiritoriparts, logo:kiritoriparts
- moved J2 5.11 mm to (189.9, 28.5), turned to 0 degrees
- moved J1 4.98 mm to (113.8, 24.0), turned to 180 degrees
Connections:
- J12 pad A: Net-(J12-PadA) -> (no net)
- J13 pad A: Net-(J13-PadA) -> (no net)
- U1 pad 11: Net-(U1-Pad11) -> (no net)
- U1 pad 13: Net-(U1-Pad13) -> (no net)
- U1 pad 15: Net-(U1-Pad15) -> (no net)
- U1 pad 19: Net-(U1-Pad19) -> (no net)
- U1 pad 20: Net-(U1-Pad20) -> (no net)
- U1 pad 24: Net-(U1-Pad24) -> (no net)
- U1 pad 5: Net-(U1-Pad5) -> (no net)
- U1 pad 6: Net-(U1-Pad6) -> (no net)
- U2 pad 11: Net-(U2-Pad11) -> (no net)
- U2 pad 13: Net-(U2-Pad13) -> (no net)
- U2 pad 15: Net-(U2-Pad15) -> (no net)
- U2 pad 19: Net-(U2-Pad19) -> (no net)
- U2 pad 20: Net-(U2-Pad20) -> (no net)
- U2 pad 24: Net-(U2-Pad24) -> (no net)
- U2 pad 5: Net-(U2-Pad5) -> (no net)
- U2 pad 6: Net-(U2-Pad6) -> (no net)
Routing:
- net col3R: track 108.2 -> 68.6 mm
- net Net-(L5-Pad1): track 32.6 -> 0.00 mm
- net Net-(L4-Pad1): track 32.2 -> 0.00 mm
- net Net-(L1-Pad1): track 24.8 -> 0.00 mm
- net Net-(L2-Pad1): track 22.9 -> 0.00 mm
- net GND: track 382.1 -> 369.0 mm
- net VCC: track 313.9 -> 326.6 mm, vias 7 -> 5
- net LEDR: track 102.2 -> 106.0 mm
- net LEDL: track 120.0 -> 117.6 mm, vias 2 -> 0
Other:
- board text added: "cool936 designed by m.ki date 20220516 ver.1.4"
- board text removed: "cool936 designed by m.ki date 20220503 ver.1.3"

Commit message: fix
Parts:
- added G***: LOGO, logo:dragonbreath_left, B.Cu at (82.1, 38.9)
- added G***: LOGO, logo:dragonbreath, B.Cu at (219.8, 39.3)
Routing:
- net col4R: track 68.3 -> 45.1 mm, vias 4 -> 2
- net GND: track 369.0 -> 358.9 mm
- net col3L: track 119.9 -> 110.0 mm
- net col2L: track 100.5 -> 90.6 mm
- net col4L: track 109.1 -> 99.3 mm
- net col0L: track 106.3 -> 96.5 mm
- net col1L: track 82.5 -> 73.2 mm
- net col1R: track 128.3 -> 121.8 mm
- net row3R: track 183.1 -> 178.1 mm, vias 5 -> 4
- net Net-(D101-Pad2): track 12.1 -> 8.83 mm
- net Net-(D22-Pad2): track 16.7 -> 13.4 mm
- net Net-(D29-Pad2): track 13.0 -> 9.69 mm
- net Net-(D302-Pad2): track 30.0 -> 26.7 mm
- net Net-(D1-Pad2): track 16.1 -> 12.8 mm
- net Net-(D301-Pad2): track 12.9 -> 9.59 mm
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Other:
- board text added: "cool936 designed by m.ki date 20220831 ver.1.51"
- board text removed: "cool936 designed by m.ki date 20220516 ver.1.4"
